File: eagle/HV ADC/CW output.sch (EAGLE design)
At the start: 5 parts, among them J1 HV, J2 ADC

Commit message: Latest CW tests
Parts:
- added R4: 270, SparkFun-Resistors:15KOHM-HORIZ-1/4W-5%
- added R5: 68, SparkFun-Resistors:15KOHM-HORIZ-1/4W-5%
Connections:
- new net 5V: R1.1, R4.1, R4.2, R5.2
- net 3.3V: now also R5.1; no longer R1.1
Other:
- note added: "CW Output 0 to -40 KV"
- note added: "~ 1.0V"
- note removed: "CW Output 40 KV"
- moved on the sheet: J2, R1
Changed lines of the file:
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@@
 <part name="J2" library="SparkFun-Connectors" library_urn="urn:adsk.eagle:library:513" deviceset="CONN_01" device="PTH_2MM" package3d_urn="urn:adsk.eagle:package:38029/1" value="ADC"/>
 <part name="R2" library="cwParts" deviceset="SM108031005FE" device="" value="HV 200M"/>
+<part name="R4" library="SparkFun-Resistors" library_urn="urn:adsk.eagle:library:532" deviceset="15KOHM" device="-HORIZ-1/4W-5%" package3d_urn="urn:adsk.eagle:package:39658/1" value="270"/>
+<part name="R5" library="SparkFun-Resistors" library_urn="urn:adsk.eagle:library:532" deviceset="15KOHM" device="-HORIZ-1/4W-5%" package3d_urn="urn:adsk.eagle:package:39658/1" value="68"/>
+<part name="SUPPLY1" library="SparkFun-PowerSymbols" library_urn="urn:adsk.eagle:library:530" deviceset="5V" device=""/>
 </parts>
 <sheets>
@@
 <plain>
 <text x="12.7" y="104.14" size="1.778" layer="91">CW Output
-40 KV</text>
+0 to -40 KV</text>
+<text x="-17.78" y="60.96" size="1.778" layer="91">~ 1.0V</text>
 </plain>
 <instances>
-<instance part="R1" gate="G$1" x="5.08" y="50.8" smashed="yes" rot="R90">
-<attribute name="NAME" x="3.556" y="50.8" size="1.778" layer="95" font="vector" rot="R90" align="bottom-center"/>
-<attribute name="VALUE" x="6.604" y="50.8" size="1.778" layer="96" font="vector" rot="R90" align="top-center"/>
+<instance part="R1" gate="G$1" x="-5.08" y="58.42" smashed="yes">
+<attribute name="NAME" x="-5.08" y="59.944" size="1.778" layer="95" font="vector" align="bottom-center"/>
+<attribute name="VALUE" x="-5.08" y="56.896" size="1.778" layer="96" font="vector" align="top-center"/>
 </instance>
 <instance part="R3" gate="G$1" x="5.08" y="78.74" smashed="yes" rot="R90">
@@
 <attribute name="VALUE" x="8.128" y="91.948" size="1.778" layer="96" rot="R270" align="center-left"/>
 </instance>
-<instance part="GND2" gate="G$1" x="5.08" y="43.18" smashed="yes">
-<attribute name="VALUE" x="5.08" y="40.386" size="1.778" layer="96" align="top-center"/>
+<instance part="GND2" gate="G$1" x="-15.24" y="43.18" smashed="yes">
+<attribute name="VALUE" x="-15.24" y="40.386" size="1.778" layer="96" align="top-center"/>
 </instance>
 <instance part="J1" gate="G$1" x="5.08" y="104.14" smashed="yes" rot="R270">
@@
 <attribute name="NAME" x="8.128" y="101.6" size="1.778" layer="95" font="vector"/>
 </instance>
-<instance part="J2" gate="G$1" x="22.86" y="58.42" smashed="yes" rot="R180">
-<attribute name="VALUE" x="24.384" y="63.5" size="1.778" layer="96" font="vector" rot="R180"/>
-<attribute name="NAME" x="23.368" y="55.118" size="1.778" layer="95" font="vector" rot="R180"/>
+<instance part="J2" gate="G$1" x="5.08" y="45.72" smashed="yes" rot="R90">
+<attribute name="VALUE" x="10.16" y="44.196" size="1.778" layer="96" font="vector" rot="R90"/>
+<attribute name="NAME" x="1.778" y="45.212" size="1.778" layer="95" font="vector" rot="R90"/>
 </instance>
 <instance part="R2" gate="G$1" x="5.08" y="60.96" smashed="yes" rot="R90">
@@
 <attribute name="VALUE" x="8.128" y="74.168" size="1.778" layer="96" rot="R270" align="center-left"/>
 </instance>
+<instance part="R4" gate="G$1" x="-22.86" y="58.42" smashed="yes">
+<attribute name="NAME" x="-22.86" y="59.944" size="1.778" layer="95" font="vector" align="bottom-center"/>
+<attribute name="VALUE" x="-22.86" y="56.896" size="1.778" layer="96" font="vector" align="top-center"/>
+</instance>
+<instance part="R5" gate="G$1" x="-15.24" y="50.8" smashed="yes" rot="R90">
+<attribute name="NAME" x="-16.764" y="50.8" size="1.778" layer="95" font="vector" rot="R90" align="bottom-center"/>
+<attribute name="VALUE" x="-13.716" y="50.8" size="1.778" layer="96" font="vector" rot="R90" align="top-center"/>
+</instance>
+<instance part="SUPPLY1" gate="G$1" x="-27.94" y="58.42" smashed="yes" rot="R90">
+<attribute name="VALUE" x="-32.766" y="59.182" size="1.778" layer="96" rot="R180" align="bottom-center"/>
+</instance>
 </instances>
 <busses>
 </busses>
 <nets>
-<net name="3.3V" class="0">
-<segment>
-<pinref part="R1" gate="G$1" pin="1"/>
-<pinref part="GND2" gate="G$1" pin="3.3V"/>
-</segment>
-</net>
 <net name="N$2" class="0">
 <segment>
@@
 </segment>
 </net>
-<net name="N$3" class="0">
+<net name="3.3V" class="0">
+<segment>
+<pinref part="R5" gate="G$1" pin="1"/>
+<pinref part="GND2" gate="G$1" pin="3.3V"/>
+</segment>
+</net>
+<net name="5V" class="0">
+<segment>
+<pinref part="R4" gate="G$1" pin="2"/>
+<pinref part="SUPPLY1" gate="G$1" pin="5V"/>
+<pinref part="R4" gate="G$1" pin="1"/>
+<pinref part="R5" gate="G$1" pin="2"/>
+<pinref part="R1" gate="G$1" pin="1"/>
+<wire x1="-15.24" y1="58.42" x2="-15.24" y2="55.88" width="0.1524" layer="91"/>
+<wire x1="-10.16" y1="58.42" x2="-15.24" y2="58.42" width="0.1524" layer="91"/>
+<wire x1="-17.78" y1="58.42" x2="-15.24" y2="58.42" width="0.1524" layer="91"/>
+<junction x="-15.24" y="58.42"/>
+</segment>
+</net>
+<net name="N$4" class="0">
 <segment>
 <pinref part="R2" gate="G$1" pin="1"/>
+<pinref part="J2" gate="G$1" pin="1"/>
+<wire x1="5.08" y1="60.96" x2="5.08" y2="58.42" width="0.1524" layer="91"/>
 <pinref part="R1" gate="G$1" pin="2"/>
-<wire x1="5.08" y1="60.96" x2="5.08" y2="58.42" width="0.1524" layer="91"/>
-<pinref part="J2" gate="G$1" pin="1"/>
-<wire x1="5.08" y1="58.42" x2="5.08" y2="55.88" width="0.1524" layer="91"/>
-<wire x1="15.24" y1="58.42" x2="5.08" y2="58.42" width="0.1524" layer="91"/>
+<wire x1="5.08" y1="58.42" x2="5.08" y2="53.34" width="0.1524" layer="91"/>
+<wire x1="0" y1="58.42" x2="5.08" y2="58.42" width="0.1524" layer="91"/>
 <junction x="5.08" y="58.42"/>
 </segment>
