File: eagle/Isolator/Isolator1.sch (EAGLE design)
At the start: 15 parts, among them J1 61300411121, J2 61300411121, J4 PJ-102A, Q1 BC557C, Q2 BC557C

Commit message: Working - check power jack
Parts:
- removed J4: PJ-102A, jack:PJ-102A
- added U$1: CUI_PJ-102A, con-dc-jack:CUI_PJ-102A
- OK1, OK2: value SFH618A-2 -> SFH617A-2
- Q1, Q2: value BC557C -> 2N3906
- R1, R2: value (none) -> 200; device SparkFun-Resistors:RESISTORAXIAL-0.3 -> resistor:R-US_0207/7
- R3, R6: value (none) -> 1500; device SparkFun-Resistors:RESISTORAXIAL-0.3 -> resistor:R-US_0207/7
- R4, R8: value (none) -> 1000; device SparkFun-Resistors:RESISTORAXIAL-0.3 -> resistor:R-US_0207/7
- R5, R7: value (none) -> 75; device SparkFun-Resistors:RESISTORAXIAL-0.3 -> resistor:R-US_0207/7
Connections:
- new net CASE: U$1.@3
- net GND2: now also U$1.VSS; no longer J4.2, J4.3
- net VCC2: now also U$1.VDD; no longer J4.1
