File: eagle/Power Dist 9/PowerDist.brd (EAGLE design)
At the start: 38.1 x 129.5 mm, 17 parts

Commit message: done
Parts:
- moved PS3 1.27 mm to (6.35, 39.4)
- moved C3 1.27 mm to (6.35, 44.5)
- moved C7 1.27 mm to (21.6, 44.5)
Routing:
- net N$9: track 0.00 -> 25.4 mm
- net N$8: track 0.00 -> 25.4 mm
- net N$7: track 0.00 -> 25.4 mm
- net N$10: track 0.00 -> 25.4 mm
- net N$5: track 0.00 -> 14.8 mm
- net N$6: track 0.00 -> 14.8 mm
- net N$4: track 0.00 -> 14.8 mm
- net N$3: track 0.00 -> 14.8 mm
Other:
- board text added: "0V"
- board text added: "24V"
- board text added: "3kV Isolated 24VDC to 9VDC 1W Regulated"
- board text added: "9V"
- board text added: "chuck@whitmer.us"
